File: JustBreathe_Electronics/JustBreathe_Electronics.kicad_pcb (KiCad board)
At the start: 2 copper layers, 78 x 56.5 mm, 17 parts, among them Q1 IRLZ34N, U1 DFR0299, U2 WEMOS_D1_mini

Commit message: generate gerber files
Parts:
- renumbered Button_Connector1 to BUTTON, PIR_Connector1 to PIR, RV1 to POT, Pump1 to PUMP, RTC_Connector1 to RTC, Speaker1 to SPEAKER
Routing:
- net GND: track 134.9 -> 137.7 mm
- net /Vcc: track 142.1 -> 141.1 mm
Other:
- board text added: "+"
- board text added: "-"
- board text added: "SDA"

Commit message: fix circuit / create design for bottle holder
Parts:
- renumbered BUTTON to Button_Connector1, PIR to PIR_Connector1, PUMP to Pump1, RTC to RTC_Connector1, POT to RV1, SPEAKER to Speaker1
Connections:
- Q1 pad 2: GND -> Net-(D1-A)
- Q1 pad 3: Net-(D1-A) -> GND
Routing:
- net GND: track 137.7 -> 148.1 mm, vias 3 -> 0
- net /Vcc: track 141.1 -> 144.4 mm, vias 3 -> 0
- net Net-(D1-A): track 24.8 -> 24.0 mm
